Commit message: improved urdf process

File: examples/robot.urdf (robot description, URDF)
Before this commit: robot simple_arm, 3 links, 2 joints
Links:
- removed link link1
- removed link link2
- added link elbow_pitch_Link, mass 0.199195477063106; collision mesh filename=package://JG0.8.0-A4-000 手臂组件J（右）_初版（URDF）.SLDASM/meshes/el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; visual mesh filename=package://JG0.8.0-A4-000 手臂组件J（右）_初版（URDF）.SLDASM/meshes/el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
- added link elbow_yaw_Link, mass 0.292862233057086; collision mesh filename=package://JG0.8.0-A4-000 手臂组件J（右）_初版（URDF）.SLDASM/meshes/el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; visual mesh filename=package://JG0.8.0-A4-000 手臂组件J（右）_初版（URDF）.SLDASM/meshes/el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
- added link shouder_yaw_Link, mass 0.698603201546955; collision mesh filename=package://JG0.8.0-A4-000 手臂组件J（右）_初版（URDF）.SLDASM/meshes/sh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; visual mesh filename=package://JG0.8.0-A4-000 手臂组件J（右）_初版（URDF）.SLDASM/meshes/sh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
- added link shoulder_pitch_Link, mass 0.586035180256861; collision mesh filename=package://JG0.8.0-A4-000 手臂组件J（右）_初版（URDF）.SLDASM/meshes/sh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; visual mesh filename=package://JG0.8.0-A4-000 手臂组件J（右）_初版（URDF）.SLDASM/meshes/sh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
- added link shoulder_roll_Link, mass 0.199195477062016; collision mesh filename=package://JG0.8.0-A4-000 手臂组件J（右）_初版（URDF）.SLDASM/meshes/sh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; visual mesh filename=package://JG0.8.0-A4-000 手臂组件J（右）_初版（URDF）.SLDASM/meshes/sh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
- added link wrist_pitch_Link, mass 0.125358654619444; collision mesh filename=package://JG0.8.0-A4-000 手臂组件J（右）_初版（URDF）.SLDASM/meshes/wr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; visual mesh filename=package://JG0.8.0-A4-000 手臂组件J（右）_初版（URDF）.SLDASM/meshes/wr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
- added link wrist_roll_Link, mass 0.158699506149188; collision mesh filename=package://JG0.8.0-A4-000 手臂组件J（右）_初版（URDF）.SLDASM/meshes/wr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; visual mesh filename=package://JG0.8.0-A4-000 手臂组件J（右）_初版（URDF）.SLDASM/meshes/wr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
- link base_link: mass 0.5 -> 0.310055800796731; geometry collision mesh filename=package://JG0.8.0-A4-000 手臂组件J（右）_初版（URDF）.SLDASM/meshes/ba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; visual mesh filename=package://JG0.8.0-A4-000 手臂组件J（右）_初版（URDF）.SLDASM/meshes/ba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
Joints:
- removed joint joint1
- removed joint joint2
- added joint joint_1: type revolute, parent base_link, child shoulder_pitch_Link, origin xyz=0 -0.1255 0 rpy=1.5708 1.5708 0, axis 0 0 -1, limit lower=0 upper=0 effort=0 velocity=0
- added joint joint_2: type revolute, parent shoulder_pitch_Link, child shoulder_roll_Link, origin xyz=0.06 0 0 rpy=1.5708 0 0, axis 0 0 -1, limit lower=0 upper=0 effort=0 velocity=0
- added joint joint_3: type revolute, parent shoulder_roll_Link, child shouder_yaw_Link, origin xyz=0 0 0 rpy=-1.5708 0 -1.5708, axis 0 0 1, limit lower=0 upper=0 effort=0 velocity=0
- added joint joint_4: type revolute, parent shouder_yaw_Link, child elbow_pitch_Link, origin xyz=0 0 0.22 rpy=3.1416 -1.5708 0, axis 0 0 1, limit lower=0 upper=0 effort=0 velocity=0
- added joint joint_5: type revolute, parent elbow_pitch_Link, child elbow_yaw_Link, origin xyz=0 0 0 rpy=-1.5708 0 -1.5708, axis 0 0 1, limit lower=0 upper=0 effort=0 velocity=0
- added joint joint_6: type revolute, parent elbow_yaw_Link, child wrist_roll_Link, origin xyz=0 0 0.22 rpy=0 -1.5708 0, axis 0 0 1, limit lower=0 upper=0 effort=0 velocity=0
- added joint joint_7: type revolute, parent wrist_roll_Link, child wrist_pitch_Link, origin xyz=0.00844 0 0 rpy=0 0 0, axis 0 -1 0, limit lower=0 upper=0 effort=0 velocity=0

Commit message: full urdf process and use trac-ik, this chain is functional

File: examples/robot.urdf (robot description, URDF)
Before this commit: robot JG0.8.0-A4-000 手臂组件J（右）_初版（URDF）.SLDASM, 8 links, 7 joints
Links:
- link base_link: geometry 
- link elbow_pitch_Link: geometry 
- link elbow_yaw_Link: geometry 
- link shouder_yaw_Link: geometry 
- link shoulder_pitch_Link: geometry 
- link shoulder_roll_Link: geometry 
- link wrist_pitch_Link: geometry 
- link wrist_roll_Link: geometry 
